File: rc2014/kicad/card/card.kicad_pcb (KiCad board)
At the start: 4 copper layers, 63.5 x 102.6 mm, 27 parts, among them J1 Conn_RC40_Male, J2 DB15_Female_HighDensity, J3 Conn_02x06_Top_Bottom, SW1 SW_DIP_x07, U1 74HCT688, U2 SN74LVC8T245PWR, U3 SN74LVC8T245PWR, U4 VDC-II

Commit message: Repin U4
Parts:
- removed J3: Conn_02x06_Top_Bottom, card:PinHeader_2x06_P2.54mm_Vertical_SMD_top_down
- removed R10, R12, R8: 270, Resistor_THT:R_Axial_DIN0207_L6.3mm_D2.5mm_P10.16mm_Horizontal
- removed R11, R13, R9: 510, Resistor_THT:R_Axial_DIN0207_L6.3mm_D2.5mm_P10.16mm_Horizontal
- added C7: C, Capacitor_THT:C_Disc_D6.0mm_W4.4mm_P5.00mm, F.Cu at (79.8, 118.9)
- J2: value DB15_Female_HighDensity -> VideoMezzanine14; footprint Connector_Dsub:DSUB-15-HD_Female_Horizontal_P2.29x1.98mm_EdgePinOffset8.35mm_Housed_MountingHolesOffset10.89mm -> Package_DIP:DIP-14_W7.62mm_Socket
- U4: value VDC-II -> VDC-II-card
- moved J2 30.9 mm to (72.4, 114.6), turned to 270 degrees
Connections:
- net Net-(J2-Pad14) renamed /R1
- J2 pad 1: Net-(J2-Pad1) -> /R2
- J2 pad 10: GNDD -> /B1
- J2 pad 11: Net-(J2-Pad11) -> +3V3
- J2 pad 12: Net-(J2-Pad12) -> /G0
- J2 pad 13: Net-(J2-Pad13) -> /G2
- J2 pad 2: Net-(J2-Pad2) -> /R0
- J2 pad 3: Net-(J2-Pad3) -> /G1
- J2 pad 4: Net-(J2-Pad4) -> GNDD
- J2 pad 5: GNDD -> /B2
- J2 pad 6: GNDD -> /B0
- J2 pad 7: GNDD -> /HSYNC
- J2 pad 8: GNDD -> /VSYNC
- U4 pad 15: Net-(J2-Pad13) -> /R2
- U4 pad 17: Net-(U4-Pad17) -> /R0
- U4 pad 18: Net-(J3-Pad3) -> /G2
- U4 pad 19: Net-(J3-Pad8) -> /G1
- U4 pad 20: Net-(U4-Pad20) -> /G0
- U4 pad 21: Net-(J3-Pad10) -> /B2
- U4 pad 22: Net-(J3-Pad2) -> /B1
- U4 pad 23: Net-(U4-Pad23) -> /B0
- U4 pad 24: Net-(J3-Pad4) -> /HSYNC
- U4 pad 25: Net-(J3-Pad9) -> /VSYNC

Commit message: Finish PCB layout for main PP board
Parts:
- C7: value C -> 100nF
- moved C7 2.18 mm to (78.5, 120.7), turned to 90 degrees
Routing:
- net +3V3: track 67.1 -> 116.4 mm, vias 0 -> 1
- net /VSYNC: track 0.00 -> 48.2 mm
- net /B1: track 0.00 -> 37.6 mm
- net /HSYNC: track 0.00 -> 36.1 mm
- net /B0: track 0.00 -> 32.5 mm
- net /G0: track 0.00 -> 30.4 mm
- net /B2: track 0.00 -> 26.3 mm
- net /G2: track 0.00 -> 24.2 mm
- net /G1: track 0.00 -> 19.2 mm
- net /R1: track 0.00 -> 18.5 mm
- net /R0: track 0.00 -> 13.0 mm
- net /R2: track 0.00 -> 7.32 mm
- net GNDD: track 20.5 -> 24.5 mm, vias 0 -> 4
- net +5V: track 1.30 -> 3.65 mm, vias 0 -> 2
- net Net-(U3-Pad7): track 19.4 -> 18.7 mm
- added copper zone on In2.Cu, net +5V
- added copper zone on In1.Cu, net GNDD
Other:
- net class Power added: clearance 0.254, trace_width 0.254, via_dia 0.4572, via_drill 0.254
- board text added: "PIXEL PUSHER REV 4A / 2020 AUG 28 / SAF2"
